Commit message: add velodyne lidar and depth cam to urdf

File: robo_base_description/urdf/robot_event_cam.urdf.xacro (robot description, xacro)
@@ -90,5 +90,5 @@
   <!-- AGV lidar -->
   <joint name="base_footprint_lidar_joint" type="fixed">
-	  <origin xyz="0.0 0.0 ${agv_base_height + box_size}" rpy="0 0 ${M_PI}" />
+	  <origin xyz="0.0 0.0 ${agv_base_height + box_size*2}" rpy="0 0 ${M_PI}" />
     <parent link="base_footprint"/>
     <child link="agv_lidar" />
@@ -131,4 +131,73 @@
     </sensor>
   </gazebo>
+  <!-- depth camera -->
+  <joint name="base_footprint_camera_joint" type="fixed">
+	  <origin xyz="${agv_base_length/2 - box_size/2} 0.0 ${agv_base_height + box_size}" rpy="0 0 0" />
+    <parent link="base_footprint"/>
+    <child link="depth_cam" />
+  </joint>
+  <link name="depth_cam">
+    <visual>
+      <origin xyz="0 0 0" rpy="0 0 0" />
+      <geometry>
+        <box size="${box_size} ${box_size} ${box_size}"/>
+      </geometry>
+      <material name="Blue" />
+    </visual>
+  </link>
+  <xacro:property name="link_name" value="depth_cam" />
+  <xacro:property name="camera_name" value="realsense" />
+  <xacro:property name="frame_name" value="depth_cam" />
+  <gazebo reference="${link_name}">
+    <material>Gazebo/Blue</material>
+    <sensor name="${link_name}_camera" type="depth">
+      <update_rate>20</update_rate>
+      <camera>
+        <horizontal_fov>1.047198</horizontal_fov>
+        <image>
+          <width>640</width>
+          <height>480</height>
+          <format>R8G8B8</format>
+        </image>
+        <clip>
+          <near>0.05</near>
+          <far>3</far>
+        </clip>
+      </camera>
+      <plugin name="${link_name}_controller" filename="libgazebo_ros_openni_kinect.so">
+        <baseline>0.2</baseline>
+        <alwaysOn>true</alwaysOn>
+        <updateRate>1.0</updateRate>
+        <cameraName>${camera_name}_ir</cameraName>
+        <imageTopicName>/${camera_name}/color/image_raw</imageTopicName>
+        <cameraInfoTopicName>/${camera_name}/color/camera_info</cameraInfoTopicName>
+        <depthImageTopicName>/${camera_name}/depth/image_raw</depthImageTopicName>
+        <depthImageInfoTopicName>/${camera_name}/depth/camera_info</depthImageInfoTopicName>
+        <pointCloudTopicName>/${camera_name}/depth/points</pointCloudTopicName>
+        <frameName>${frame_name}</frameName>
+        <pointCloudCutoff>0.5</pointCloudCutoff>
+        <pointCloudCutoffMax>3.0</pointCloudCutoffMax>
+        <distortionK1>0.00000001</distortionK1>
+        <distortionK2>0.00000001</distortionK2>
+        <distortionK3>0.00000001</distortionK3>
+        <distortionT1>0.00000001</distortionT1>
+        <distortionT2>0.00000001</distortionT2>
+        <CxPrime>0</CxPrime>
+        <Cx>0</Cx>
+        <Cy>0</Cy>
+        <focalLength>0</focalLength>
+        <hackBaseline>0</hackBaseline>
+      </plugin>
+    </sensor>
+  </gazebo>
+  <!-- Veldoyne Lidar  -->
+  <xacro:arg name="gpu" default="false"/>
+  <xacro:property name="gpu" value="$(arg gpu)" />
+  <xacro:arg name="organize_cloud" default="false"/>
+  <xacro:property name="organize_cloud" value="$(arg organize_cloud)" />
+  <xacro:include filename="$(find velodyne_description)/urdf/VLP-16.urdf.xacro"/>
+  <xacro:VLP-16 parent="base_footprint" name="velodyne" topic="/velodyne_points" organize_cloud="${organize_cloud}" hz="10" samples="440" gpu="${gpu}">
+    <origin xyz="0.0 0.0 ${agv_base_height+box_size}" rpy="0 0 0" />
+  </xacro:VLP-16>
   <gazebo>
     <!-- <plugin name="differential_drive_controller" filename="libgazebo_ros_diff_drive.so"> -->

Commit message: set correct frame id for depth cam

File: robo_base_description/urdf/robot_event_cam.urdf.xacro (robot description, xacro)
@@ -146,7 +146,13 @@
     </visual>
   </link>
+  <joint name="cam_frame_id_joint" type="fixed">
+	  <origin xyz="0 0.0 0" rpy="${-M_PI_2} 0 ${-M_PI_2}" />
+    <parent link="depth_cam"/>
+    <child link="cam_frame_id" />
+  </joint>
+  <link name="cam_frame_id"/>
   <xacro:property name="link_name" value="depth_cam" />
   <xacro:property name="camera_name" value="realsense" />
-  <xacro:property name="frame_name" value="depth_cam" />
+  <xacro:property name="frame_name" value="cam_frame_id" />
   <gazebo reference="${link_name}">
     <material>Gazebo/Blue</material>

Commit message: add 3d lidar and depth cam to description

File: robo_base_description/urdf/robot_event_cam.urdf.xacro (robot description, xacro)
@@ -90,5 +90,5 @@
   <!-- AGV lidar -->
   <joint name="base_footprint_lidar_joint" type="fixed">
-	  <origin xyz="0.0 0.0 ${agv_base_height + box_size*2}" rpy="0 0 ${M_PI}" />
+	  <origin xyz="0.0 0.0 ${agv_base_height + box_size*2}" rpy="0 0 0" />
     <parent link="base_footprint"/>
     <child link="agv_lidar" />
@@ -132,64 +132,90 @@
   </gazebo>
   <!-- depth camera -->
+  <xacro:property name="r200_cam_rgb_px" value="0.005"/>
+  <xacro:property name="r200_cam_rgb_py" value="0.018"/>
+  <xacro:property name="r200_cam_rgb_pz" value="0.013"/>
+  <xacro:property name="r200_cam_depth_offset" value="0.01"/>
+  <xacro:arg name="camera_visual" default="false"/>
   <joint name="base_footprint_camera_joint" type="fixed">
 	  <origin xyz="${agv_base_length/2 - box_size/2} 0.0 ${agv_base_height + box_size}" rpy="0 0 0" />
     <parent link="base_footprint"/>
-    <child link="depth_cam" />
-  </joint>
-  <link name="depth_cam">
+    <child link="camera_link" />
+  </joint>
+  <link name="camera_link">
     <visual>
-      <origin xyz="0 0 0" rpy="0 0 0" />
-      <geometry>
-        <box size="${box_size} ${box_size} ${box_size}"/>
-      </geometry>
-      <material name="Blue" />
-    </visual>
-  </link>
-  <joint name="cam_frame_id_joint" type="fixed">
-	  <origin xyz="0 0.0 0" rpy="${-M_PI_2} 0 ${-M_PI_2}" />
-    <parent link="depth_cam"/>
-    <child link="cam_frame_id" />
-  </joint>
-  <link name="cam_frame_id"/>
-  <xacro:property name="link_name" value="depth_cam" />
-  <xacro:property name="camera_name" value="realsense" />
-  <xacro:property name="frame_name" value="cam_frame_id" />
-  <gazebo reference="${link_name}">
-    <material>Gazebo/Blue</material>
-    <sensor name="${link_name}_camera" type="depth">
-      <update_rate>20</update_rate>
+     <origin xyz="0 0 0" rpy="1.57 0 1.57"/>
+      <geometry>
+       <mesh filename="package://turtlebot3_description/meshes/sensors/r200.dae" />
+      </geometry>
+    </visual>
+    <collision>
+      <origin xyz="0.003 0.065 0.007" rpy="0 0 0"/>
+      <geometry>
+        <box size="0.012 0.132 0.020"/>
+      </geometry>
+    </collision>
+  </link>
+  <joint name="camera_rgb_joint" type="fixed">
+    <origin xyz="${r200_cam_rgb_px} ${r200_cam_rgb_py} ${r200_cam_rgb_pz}" rpy="0 0 0"/>
+    <parent link="camera_link"/>
+    <child link="camera_rgb_frame"/>
+  </joint>
+  <link name="camera_rgb_frame"/>
+  <joint name="camera_rgb_optical_joint" type="fixed">
+    <origin xyz="0 0 0" rpy="-1.57 0 -1.57"/>
+    <parent link="camera_rgb_frame"/>
+    <child link="camera_rgb_optical_frame"/>
+  </joint>
+  <link name="camera_rgb_optical_frame"/>
+  <joint name="camera_depth_joint" type="fixed">
+    <origin xyz="${r200_cam_rgb_px} ${r200_cam_rgb_py + r200_cam_depth_offset} ${r200_cam_rgb_pz}" rpy="0 0 0"/>
+    <parent link="camera_link"/>
+    <child link="camera_depth_frame"/>
+  </joint>
+  <link name="camera_depth_frame"/>
+  <joint name="camera_depth_optical_joint" type="fixed">
+    <origin xyz="0 0 0" rpy="-1.57 0 -1.57"/>
+    <parent link="camera_depth_frame"/>
+    <child link="camera_depth_optical_frame"/>
+  </joint>
+  <link name="camera_depth_optical_frame"/>
+  <gazebo reference="camera_rgb_frame">
+    <sensor type="depth" name="realsense_R200">
+      <always_on>true</always_on>
+      <visualize>$(arg camera_visual)</visualize>
       <camera>
-        <horizontal_fov>1.047198</horizontal_fov>
-        <image>
-          <width>640</width>
-          <height>480</height>
-          <format>R8G8B8</format>
-        </image>
-        <clip>
-          <near>0.05</near>
-          <far>3</far>
-        </clip>
+          <horizontal_fov>1.3439</horizontal_fov>
+          <image>
+              <width>1920</width>
+              <height>1080</height>
+              <format>R8G8B8</format>
+          </image>
+          <depth_camera></depth_camera>
+          <clip>
+              <near>0.03</near>
+              <far>100</far>
+          </clip>
       </camera>
-      <plugin name="${link_name}_controller" filename="libgazebo_ros_openni_kinect.so">
+      <plugin name="camera_controller" filename="libgazebo_ros_openni_kinect.so">
         <baseline>0.2</baseline>
         <alwaysOn>true</alwaysOn>
-        <updateRate>1.0</updateRate>
-        <cameraName>${camera_name}_ir</cameraName>
-        <imageTopicName>/${camera_name}/color/image_raw</imageTopicName>
-        <cameraInfoTopicName>/${camera_name}/color/camera_info</cameraInfoTopicName>
-        <depthImageTopicName>/${camera_name}/depth/image_raw</depthImageTopicName>
-        <depthImageInfoTopicName>/${camera_name}/depth/camera_info</depthImageInfoTopicName>
-        <pointCloudTopicName>/${camera_name}/depth/points</pointCloudTopicName>
-        <frameName>${frame_name}</frameName>
-        <pointCloudCutoff>0.5</pointCloudCutoff>
-        <pointCloudCutoffMax>3.0</pointCloudCutoffMax>
-        <distortionK1>0.00000001</distortionK1>
-        <distortionK2>0.00000001</distortionK2>
-        <distortionK3>0.00000001</distortionK3>
-        <distortionT1>0.00000001</distortionT1>
-        <distortionT2>0.00000001</distortionT2>
-        <CxPrime>0</CxPrime>
-        <Cx>0</Cx>
-        <Cy>0</Cy>
+        <updateRate>30.0</updateRate>
+        <cameraName>camera</cameraName>
+        <frameName>camera_rgb_optical_frame</frameName>
+        <imageTopicName>rgb/image_raw</imageTopicName>
+        <depthImageTopicName>depth/image_raw</depthImageTopicName>
+        <pointCloudTopicName>depth/points</pointCloudTopicName>
+        <cameraInfoTopicName>rgb/camera_info</cameraInfoTopicName>
+        <depthImageCameraInfoTopicName>depth/camera_info</depthImageCameraInfoTopicName>
+        <pointCloudCutoff>0.4</pointCloudCutoff>
+            <hackBaseline>0.07</hackBaseline>
+            <distortionK1>0.0</distortionK1>
+            <distortionK2>0.0</distortionK2>
+            <distortionK3>0.0</distortionK3>
+            <distortionT1>0.0</distortionT1>
+            <distortionT2>0.0</distortionT2>
+        <CxPrime>0.0</CxPrime>
+        <Cx>0.0</Cx>
+        <Cy>0.0</Cy>
         <focalLength>0</focalLength>
         <hackBaseline>0</hackBaseline>

Commit message: add imu to description

File: robo_base_description/urdf/robot_event_cam.urdf.xacro (robot description, xacro)
@@ -88,4 +88,47 @@
     </collision>
   </link>
+  <!-- IMU -->
+  <xacro:arg name="imu_visual"    default="true"/>
+  <joint name="imu_joint" type="fixed">
+    <parent link="agv_base_link"/>
+    <child link="imu_link"/>
+    <origin xyz="0.0 0 0.05" rpy="0 0 0"/>
+  </joint>
+  <link name="imu_link"/>
+  <gazebo reference="imu_link">
+    <sensor type="imu" name="imu">
+      <always_on>true</always_on>
+      <visualize>$(arg imu_visual)</visualize>
+    </sensor>
+    <material>Gazebo/Grey</material>
+  </gazebo>
+  <gazebo>
+    <plugin name="imu_plugin" filename="libgazebo_ros_imu.so">
+      <alwaysOn>true</alwaysOn>
+      <bodyName>imu_link</bodyName>
+      <frameName>imu_link</frameName>
+      <topicName>imu</topicName>
+      <serviceName>imu_service</serviceName>
+      <gaussianNoise>0.0</gaussianNoise>
+      <updateRate>20</updateRate>
+      <imu>
+        <noise>
+          <type>gaussian</type>
+          <rate>
+            <mean>0.0</mean>
+            <stddev>2e-4</stddev>
+            <bias_mean>0.0000075</bias_mean>
+            <bias_stddev>0.0000008</bias_stddev>
+          </rate>
+          <accel>
+            <mean>0.0</mean>
+            <stddev>1.7e-2</stddev>
+            <bias_mean>0.1</bias_mean>
+            <bias_stddev>0.001</bias_stddev>
+          </accel>
+        </noise>
+      </imu>
+    </plugin>
+  </gazebo>
   <!-- AGV lidar -->
   <joint name="base_footprint_lidar_joint" type="fixed">
